Commit message: prueba con ejes

File: src/rover_description/robots/robot.urdf.xacro (robot description, xacro)
@@ -23,6 +23,5 @@
 <!-- Gazebo ROS control plugins -->
 <xacro:include filename="$(find rover_description)/urdf/ros2_control.urdf.xacro"/>
-<xacro:arg name="config_controllers" default="$(find gz_ros2_control_demos)/config/diff_drive_controller.yaml"/>
-<xacro:arg name="config_controllers" default="$(find rovver_description)/config/rover_controllers.yaml"/>
+<xacro:arg name="config_controllers" default="$(find rover_description)/config/robot_controllers.yaml"/>
 <xacro:arg name="update_rate" default="100"/>
 <xacro:ros2_control/>

File: src/rover_description/urdf/ros2_control.urdf.xacro (robot description, xacro)
@@ -2,74 +2,52 @@
 <robot xmlns:xacro="http://wiki.ros.org/xacro">
   <xacro:macro name="ros2_control">
-      <gazebo>
-        <plugin filename="libgz_ros2_control-system.so" name="gz_ros2_control::GazeboSimROS2ControlPlugin">
-          <parameters>$(arg config_controllers)</parameters>
-        </plugin>
-        <plugin
-          filename="gz-sim-odometry-publisher-system"
-          name="gz::sim::systems::OdometryPublisher">
-          <odom_frame>odom_gt</odom_frame>
-          <robot_base_frame>base_link</robot_base_frame>
-        </plugin>
-      </gazebo>
-      <ros2_control name="rover_interface" type="system">
-        <hardware>
-           <plugin>gz_ros2_control/GazeboSimSystem</plugin>
-        </hardware>
-        <joint name="front_left_wheel_link_joint">
-          <command_interface name="velocity">
-            <param name="min">-10</param>
-            <param name="max">10</param>
-          </command_interface>
-          <state_interface name="position"/>
-          <state_interface name="velocity"/>
-          <state_interface name="effort"/>
-        </joint>
-        <joint name="front_right_wheel_link_joint">
-          <command_interface name="velocity">
-            <param name="min">-10</param>
-            <param name="max">10</param>
-          </command_interface>
-          <state_interface name="position"/>
-          <state_interface name="velocity"/>
-          <state_interface name="effort"/>
-        </joint>
-        <joint name="back_left_wheel_link_joint">
-          <command_interface name="velocity">
-            <param name="min">-10</param>
-            <param name="max">10</param>
-          </command_interface>
-          <state_interface name="position"/>
-          <state_interface name="velocity"/>
-          <state_interface name="effort"/>
-        </joint>
-        <joint name="back_right_wheel_link_joint">
-          <command_interface name="velocity">
-            <param name="min">-10</param>
-            <param name="max">10</param>
-          </command_interface>
-          <state_interface name="position"/>
-          <state_interface name="velocity"/>
-          <state_interface name="effort"/>
-        </joint>
-        <joint name="mid_left_wheel_link_joint">
-          <command_interface name="velocity">
-            <param name="min">-10</param>
-            <param name="max">10</param>
-          </command_interface>
-          <state_interface name="position"/>
-          <state_interface name="velocity"/>
-          <state_interface name="effort"/>
-        </joint>
-        <joint name="mid_right_wheel_link_joint">
-          <command_interface name="velocity">
-            <param name="min">-10</param>
-            <param name="max">10</param>
-          </command_interface>
-          <state_interface name="position"/>
-          <state_interface name="velocity"/>
-          <state_interface name="effort"/>
-        </joint>
-      </ros2_control>
+    <gazebo>
+      <plugin
+        filename="gz_ros2_control-system"
+        name="gz_ros2_control::GazeboSimROS2ControlPlugin">
+        <parameters>$(arg config_controllers)</parameters>
+      </plugin>
+      <plugin
+        filename="gz-sim-odometry-publisher-system"
+        name="gz::sim::systems::OdometryPublisher">
+        <odom_frame>odom_gt</odom_frame>
+        <robot_base_frame>base_link</robot_base_frame>
+      </plugin>
+    </gazebo>
+    <ros2_control name="GazeboSystem" type="system">
+      <hardware>
+        <plugin>gz_ros2_control/GazeboSimSystem</plugin>
+      </hardware>
+      <joint name="front_left_wheel_link_joint">
+        <command_interface name="velocity"/>
+        <state_interface name="position"/>
+        <state_interface name="velocity"/>
+      </joint>
+      <joint name="mid_left_wheel_link_joint">
+        <command_interface name="velocity"/>
+        <state_interface name="position"/>
+        <state_interface name="velocity"/>
+      </joint>
+      <joint name="back_left_wheel_link_joint">
+        <command_interface name="velocity"/>
+        <state_interface name="position"/>
+        <state_interface name="velocity"/>
+      </joint>
+      <joint name="front_right_wheel_link_joint">
+        <command_interface name="velocity"/>
+        <state_interface name="position"/>
+        <state_interface name="velocity"/>
+      </joint>
+      <joint name="mid_right_wheel_link_joint">
+        <command_interface name="velocity"/>
+        <state_interface name="position"/>
+        <state_interface name="velocity"/>
+      </joint>
+      <joint name="back_right_wheel_link_joint">
+        <command_interface name="velocity"/>
+        <state_interface name="position"/>
+        <state_interface name="velocity"/>
+      </joint>
+    </ros2_control>
   </xacro:macro>
 </robot>
