Commit message: prueba con ejes

File: src/rover_description/urdf/wheels/rover_wheels.urdf.xacro (robot description, xacro)
@@ -1,340 +1,260 @@
 <?xml version="1.0"?>
 <robot name="arm_gripper" xmlns:xacro="http://wiki.ros.org/xacro">
-    <xacro:macro name="rover_wheels" params="parent">
+  <xacro:macro name="rover_wheels" params="parent">
     <xacro:property name="mesh_path" value="file://$(find rover_description)/meshes/dae"/>
     <joint name="axis_left_link_joint" type="fixed">
-        <origin rpy="1.60974 -0.01480 -0.06763" xyz="-0.35085 -0.70000 -0.47400"/>
-        <parent link="body_link"/>
-        <child link="axis_left_link"/>
-        <axis xyz="0.00000 0.00000 1.00000"/>
+      <origin rpy="1.60974 -0.01480 -0.06763" xyz="-0.35085 -0.70000 -0.47400"/>
+      <parent link="body_link"/>
+      <child link="axis_left_link"/>
     </joint>
     <joint name="axis_right_link_joint" type="fixed">
-        <origin rpy="-1.57080 0.00000 -0.02477" xyz="-0.35085 0.70000 -0.47400"/>
-        <parent link="body_link"/>
-        <child link="axis_right_link"/>
-        <axis xyz="0.00000 0.00000 1.00000"/>
+      <origin rpy="-1.57080 0.00000 -0.02477" xyz="-0.35085 0.70000 -0.47400"/>
+      <parent link="body_link"/>
+      <child link="axis_right_link"/>
     </joint>
     <joint name="back_left_wheel_link_joint" type="continuous">
-        <limit effort="50.0" velocity="20.00"/>
-        <origin rpy="-0.03655 0.06700 -0.01743" xyz="-1.43329 -0.48979 0.41533"/>
-        <parent link="axis_left_link"/>
-        <child link="back_left_wheel_link"/>
-        <axis xyz="0.00000 0.00000 1.00000"/>
+      <limit effort="50.0" velocity="20.00"/>
+      <origin rpy="-0.03655 0.06700 -0.01743" xyz="-1.43329 -0.48979 0.41533"/>
+      <parent link="axis_left_link"/>
+      <child link="back_left_wheel_link"/>
+      <axis xyz="0.00000 0.00000 1.00000"/>
     </joint>
     <joint name="front_left_wheel_link_joint" type="continuous">
-        <limit effort="50.0" velocity="20.00"/>
-        <origin rpy="-0.03655 0.06700 -0.01743" xyz="1.55952 -0.54195 0.21447"/>
-        <parent link="axis_left_link"/>
-        <child link="front_left_wheel_link"/>
-        <axis xyz="0.00000 0.00000 1.00000"/>
+      <limit effort="50.0" velocity="20.00"/>
+      <origin rpy="-0.03655 0.06700 -0.01743" xyz="1.55952 -0.54195 0.21447"/>
+      <parent link="axis_left_link"/>
+      <child link="front_left_wheel_link"/>
+      <axis xyz="0.00000 0.00000 1.00000"/>
     </joint>
     <joint name="mid_left_wheel_link_joint" type="continuous">
-        <limit effort="50.0" velocity="20.00"/>
-        <origin rpy="-0.03655 0.06700 -0.01743" xyz="0.06311 -0.51587 0.31490"/>
-        <parent link="axis_left_link"/>
-        <child link="mid_left_wheel_link"/>
-        <axis xyz="0.00000 0.00000 1.00000"/>
+      <limit effort="50.0" velocity="20.00"/>
+      <origin rpy="-0.03655 0.06700 -0.01743" xyz="0.06311 -0.51587 0.31490"/>
+      <parent link="axis_left_link"/>
+      <child link="mid_left_wheel_link"/>
+      <axis xyz="0.00000 0.00000 1.00000"/>
     </joint>
     <joint name="back_right_wheel_link_joint" type="continuous">
-        <limit effort="50.0" velocity="20.00"/>
-        <origin rpy="3.14159 -0.02477 -0.00000" xyz="-1.45614 0.52600 0.26402"/>
-        <parent link="axis_right_link"/>
-        <child link="back_right_wheel_link"/>
-        <axis xyz="0.00000 0.00000 1.00000"/>
+      <limit effort="50.0" velocity="20.00"/>
+      <origin rpy="3.14159 -0.02477 -0.00000" xyz="-1.45614 0.52600 0.26402"/>
+      <parent link="axis_right_link"/>
+      <child link="back_right_wheel_link"/>
+      <axis xyz="0.00000 0.00000 1.00000"/>
     </joint>
     <joint name="front_right_wheel_link_joint" type="continuous">
-        <limit effort="50.0" velocity="20.00"/>
-        <origin rpy="3.14159 -0.02477 -0.00000" xyz="1.54294 0.52600 0.33832"/>
-        <parent link="axis_right_link"/>
-        <child link="front_right_wheel_link"/>
-        <axis xyz="0.00000 0.00000 1.00000"/>
+      <limit effort="50.0" velocity="20.00"/>
+      <origin rpy="3.14159 -0.02477 -0.00000" xyz="1.54294 0.52600 0.33832"/>
+      <parent link="axis_right_link"/>
+      <child link="front_right_wheel_link"/>
+      <axis xyz="0.00000 0.00000 1.00000"/>
     </joint>
     <joint name="mid_right_wheel_link_joint" type="continuous">
-        <limit effort="50.0" velocity="20.00"/>
-        <origin rpy="3.14159 -0.02477 -0.00000" xyz="0.04340 0.52600 0.30117"/>
-        <parent link="axis_right_link"/>
-        <child link="mid_right_wheel_link"/>
-        <axis xyz="0.00000 0.00000 1.00000"/>
+      <limit effort="50.0" velocity="20.00"/>
+      <origin rpy="3.14159 -0.02477 -0.00000" xyz="0.04340 0.52600 0.30117"/>
+      <parent link="axis_right_link"/>
+      <child link="mid_right_wheel_link"/>
+      <axis xyz="0.00000 0.00000 1.00000"/>
     </joint>
     <link name="back_left_wheel_link">
-        <collision name="back_left_wheel_collision">
-            <origin rpy="-0.00497 -0.00000 0.00000" xyz="-0.00000 0.00042 -0.12869"/>
-            <geometry>
-                <mesh filename="${mesh_path}/Torus.005.dae" scale="0.40000 0.40000 0.70000"/>
-            </geometry>
-        </collision>
-        <inertial>
-            <inertia ixx="0.19403" ixy="-0.00000" ixz="0.00000" iyy="0.35189" iyz="-0.00000" izz="0.19403"/>
-            <origin rpy="0.00000 0.00000 0.00000" xyz="-0.00000 0.00042 -0.12869"/>
-            <mass value="3.00000"/>
-        </inertial>
-        <visual name="back_left_wheel">
-            <material name="Material.003"/>
-            <origin rpy="-0.00249 -0.00000 0.00000" xyz="-0.00000 0.00042 -0.12869"/>
-            <geometry>
-                <mesh filename="${mesh_path}/Torus.005.dae" scale="0.40000 0.40000 0.70000"/>
-            </geometry>
-        </visual>
+      <collision name="back_left_wheel_collision">
+        <origin rpy="-0.00497 -0.00000 0.00000" xyz="-0.00000 0.00042 -0.12869"/>
+        <geometry>
+          <mesh filename="${mesh_path}/Torus.005.dae" scale="0.40000 0.40000 0.70000"/>
+        </geometry>
+      </collision>
+      <inertial>
+        <inertia ixx="0.19403" ixy="-0.00000" ixz="0.00000" iyy="0.35189" iyz="-0.00000" izz="0.19403"/>
+        <origin rpy="0.00000 0.00000 0.00000" xyz="-0.00000 0.00042 -0.12869"/>
+        <mass value="3.00000"/>
+      </inertial>
+      <visual name="back_left_wheel">
+        <material name="Material.003"/>
+        <origin rpy="-0.00249 -0.00000 0.00000" xyz="-0.00000 0.00042 -0.12869"/>
+        <geometry>
+          <mesh filename="${mesh_path}/Torus.005.dae" scale="0.40000 0.40000 0.70000"/>
+        </geometry>
+      </visual>
     </link>
     <link name="front_left_wheel_link">
-        <collision name="front_left_wheel_collision">
-            <origin rpy="-0.00497 -0.00000 0.00000" xyz="0.00000 0.00043 -0.12796"/>
-            <geometry>
-                <mesh filename="${mesh_path}/Torus.009.dae" scale="0.40000 0.40000 0.70000"/>
-            </geometry>
-        </collision>
-        <inertial>
-            <inertia ixx="0.19403" ixy="-0.00000" ixz="0.00000" iyy="0.35189" iyz="-0.00000" izz="0.19403"/>
-            <origin rpy="0.00000 0.00000 0.00000" xyz="0.00000 0.00043 -0.12796"/>
-            <mass value="3.00000"/>
-        </inertial>
-        <visual name="front_left_wheel">
-            <material name="wheels"/>
-            <origin rpy="-0.00249 -0.00000 0.00000" xyz="0.00000 0.00043 -0.12796"/>
-            <geometry>
-                <mesh filename="${mesh_path}/Torus.009.dae" scale="0.40000 0.40000 0.70000"/>
-            </geometry>
-        </visual>
+      <collision name="front_left_wheel_collision">
+        <origin rpy="-0.00497 -0.00000 0.00000" xyz="0.00000 0.00043 -0.12796"/>
+        <geometry>
+          <mesh filename="${mesh_path}/Torus.009.dae" scale="0.40000 0.40000 0.70000"/>
+        </geometry>
+      </collision>
+      <inertial>
+        <inertia ixx="0.19403" ixy="-0.00000" ixz="0.00000" iyy="0.35189" iyz="-0.00000" izz="0.19403"/>
+        <origin rpy="0.00000 0.00000 0.00000" xyz="0.00000 0.00043 -0.12796"/>
+        <mass value="3.00000"/>
+      </inertial>
+      <visual name="front_left_wheel">
+        <material name="wheels"/>
+        <origin rpy="-0.00249 -0.00000 0.00000" xyz="0.00000 0.00043 -0.12796"/>
+        <geometry>
+          <mesh filename="${mesh_path}/Torus.009.dae" scale="0.40000 0.40000 0.70000"/>
+        </geometry>
+      </visual>
     </link>
     <link name="mid_left_wheel_link">
-        <collision name="mid_left_wheel_collision">
-            <origin rpy="-0.00497 -0.00000 0.00000" xyz="0.00000 0.00042 -0.12869"/>
-            <geometry>
-                <mesh filename="${mesh_path}/Torus.006.dae" scale="0.40000 0.40000 0.70000"/>
-            </geometry>
-            </collision>
-        <inertial>
-            <inertia ixx="0.19403" ixy="-0.00000" ixz="0.00000" iyy="0.35189" iyz="-0.00000" izz="0.19403"/>
-            <origin rpy="0.00000 0.00000 0.00000" xyz="0.00000 0.00042 -0.12869"/>
-            <mass value="3.00000"/>
-        </inertial>
-        <visual name="mid_left_wheel">
-            <material name="Material.004"/>
-            <origin rpy="-0.00249 -0.00000 0.00000" xyz="0.00000 0.00042 -0.12869"/>
-            <geometry>
-                <mesh filename="${mesh_path}/Torus.006.dae" scale="0.40000 0.40000 0.70000"/>
-            </geometry>
-        </visual>
+      <collision name="mid_left_wheel_collision">
+        <origin rpy="-0.00497 -0.00000 0.00000" xyz="0.00000 0.00042 -0.12869"/>
+        <geometry>
+          <mesh filename="${mesh_path}/Torus.006.dae" scale="0.40000 0.40000 0.70000"/>
+        </geometry>
+      </collision>
+      <inertial>
+        <inertia ixx="0.19403" ixy="-0.00000" ixz="0.00000" iyy="0.35189" iyz="-0.00000" izz="0.19403"/>
+        <origin rpy="0.00000 0.00000 0.00000" xyz="0.00000 0.00042 -0.12869"/>
+        <mass value="3.00000"/>
+      </inertial>
+      <visual name="mid_left_wheel">
+        <material name="Material.004"/>
+        <origin rpy="-0.00249 -0.00000 0.00000" xyz="0.00000 0.00042 -0.12869"/>
+        <geometry>
+          <mesh filename="${mesh_path}/Torus.006.dae" scale="0.40000 0.40000 0.70000"/>
+        </geometry>
+      </visual>
     </link>
     <link name="back_right_wheel_link">
-        <collision name="back_right_wheel_collision">
-            <origin rpy="-3.14159 0.00000 0.00000" xyz="-0.00000 0.00000 0.10000"/>
-            <geometry>
-                <mesh filename="${mesh_path}/Torus.dae" scale="0.40000 0.40000 0.70000"/>
-            </geometry>
-        </collision>
-        <inertial>
-            <inertia ixx="0.19403" ixy="0.00000" ixz="0.00000" iyy="0.35189" iyz="-0.00000" izz="0.19403"/>
-            <origin rpy="0.00000 0.00000 0.00000" xyz="-0.00000 0.00000 0.10000"/>
-            <mass value="3.00000"/>
-        </inertial>
-        <visual name="back_right_wheel">
-            <material name="Material.002"/>
-            <origin rpy="-0.00000 0.00000 0.00000" xyz="-0.00000 0.00000 0.10000"/>
-            <geometry>
-                <mesh filename="${mesh_path}/Torus.dae" scale="0.40000 0.40000 0.70000"/>
-            </geometry>
-        </visual>
+      <collision name="back_right_wheel_collision">
+        <origin rpy="-3.14159 0.00000 0.00000" xyz="-0.00000 0.00000 0.10000"/>
+        <geometry>
+          <mesh filename="${mesh_path}/Torus.dae" scale="0.40000 0.40000 0.70000"/>
+        </geometry>
+      </collision>
+      <inertial>
+        <inertia ixx="0.19403" ixy="0.00000" ixz="0.00000" iyy="0.35189" iyz="-0.00000" izz="0.19403"/>
+        <origin rpy="0.00000 0.00000 0.00000" xyz="-0.00000 0.00000 0.10000"/>
+        <mass value="3.00000"/>
+      </inertial>
+      <visual name="back_right_wheel">
+        <material name="Material.002"/>
+        <origin rpy="-0.00000 0.00000 0.00000" xyz="-0.00000 0.00000 0.10000"/>
+        <geometry>
+          <mesh filename="${mesh_path}/Torus.dae" scale="0.40000 0.40000 0.70000"/>
+        </geometry>
+      </visual>
     </link>
     <link name="front_right_wheel_link">
-        <collision name="front_right_wheel_collision">
-            <origin rpy="-3.14159 0.00000 0.00000" xyz="0.00000 0.00000 0.10000"/>
-            <geometry>
-                <mesh filename="${mesh_path}/Torus.008.dae" scale="0.40000 0.40000 0.70000"/>
-            </geometry>
-            </collision>
-        <inertial>
-            <inertia ixx="0.19403" ixy="0.00000" ixz="0.00000" iyy="0.35189" iyz="-0.00000" izz="0.19403"/>
-            <origin rpy="0.00000 0.00000 0.00000" xyz="-0.00000 0.00000 0.10000"/>
-            <mass value="3.00000"/>
-        </inertial>
-        <visual name="front_right_wheel">
-            <material name="Material"/>
-            <origin rpy="-0.00000 0.00000 0.00000" xyz="0.00000 0.00000 0.10000"/>
-            <geometry>
-                <mesh filename="${mesh_path}/Torus.008.dae" scale="0.40000 0.40000 0.70000"/>
-            </geometry>
-        </visual>
+      <collision name="front_right_wheel_collision">
+        <origin rpy="-3.14159 0.00000 0.00000" xyz="0.00000 0.00000 0.10000"/>
+        <geometry>
+          <mesh filename="${mesh_path}/Torus.008.dae" scale="0.40000 0.40000 0.70000"/>
+        </geometry>
+      </collision>
+      <inertial>
+        <inertia ixx="0.19403" ixy="0.00000" ixz="0.00000" iyy="0.35189" iyz="-0.00000" izz="0.19403"/>
+        <origin rpy="0.00000 0.00000 0.00000" xyz="-0.00000 0.00000 0.10000"/>
+        <mass value="3.00000"/>
+      </inertial>
+      <visual name="front_right_wheel">
+        <material name="Material"/>
+        <origin rpy="-0.00000 0.00000 0.00000" xyz="0.00000 0.00000 0.10000"/>
+        <geometry>
+          <mesh filename="${mesh_path}/Torus.008.dae" scale="0.40000 0.40000 0.70000"/>
+        </geometry>
+      </visual>
     </link>
     <link name="mid_right_wheel_link">
-        <collision name="mid_right_wheel_collision">
-            <origin rpy="-3.14159 0.00000 0.00000" xyz="-0.00000 0.00000 0.11498"/>
-            <geometry>
-                <mesh filename="${mesh_path}/Torus.007.dae" scale="0.40000 0.40000 0.70000"/>
-            </geometry>
-        </collision>
-        <inertial>
-            <inertia ixx="0.19403" ixy="0.00000" ixz="0.00000" iyy="0.35189" iyz="-0.00000" izz="0.19403"/>
-            <origin rpy="0.00000 0.00000 0.00000" xyz="-0.00000 0.00000 0.10000"/>
-            <mass value="3.00000"/>
-        </inertial>
-        <visual name="mid_right_wheel">
-            <material name="Material.001"/>
-            <origin rpy="-0.00000 0.00000 0.00000" xyz="-0.00000 0.00000 0.10000"/>
-            <geometry>
-                <mesh filename="${mesh_path}/Torus.007.dae" scale="0.40000 0.40000 0.70000"/>
-            </geometry>
-        </visual>
-    </link>
-      <link name="axis_left_link">
-    <collision name="axis_left_collision">
-      <origin rpy="-1.55093 0.07494 0.77002" xyz="-0.01304 0.01116 -0.07670"/>
-      <geometry>
-        <mesh filename="${mesh_path}/Cube.005.dae" scale="0.95000 0.05000 0.10000"/>
-      </geometry>
-    </collision>
-    <inertial>
-      <inertia ixx="0.00100" ixy="-0.00000" ixz="-0.00000" iyy="0.00100" iyz="0.00000" izz="0.00100"/>
-      <origin rpy="0.00000 0.00000 0.00000" xyz="0.00000 -0.00000 0.00000"/>
-      <mass value="3.00000"/>
-    </inertial>
-    <visual name="axis_left">
-      <material name="orange"/>
-      <origin rpy="-1.55093 0.07494 0.77002" xyz="-0.00365 -0.00204 -0.05382"/>
-      <geometry>
-        <mesh filename="${mesh_path}/Cube.005.dae" scale="0.95000 0.05000 0.10000"/>
-      </geometry>
-    </visual>
-  </link>
+      <collision name="mid_right_wheel_collision">
+        <origin rpy="-3.14159 0.00000 0.00000" xyz="-0.00000 0.00000 0.11498"/>
+        <geometry>
+          <mesh filename="${mesh_path}/Torus.007.dae" scale="0.40000 0.40000 0.70000"/>
+        </geometry>
+      </collision>
+      <inertial>
+        <inertia ixx="0.19403" ixy="0.00000" ixz="0.00000" iyy="0.35189" iyz="-0.00000" izz="0.19403"/>
+        <origin rpy="0.00000 0.00000 0.00000" xyz="-0.00000 0.00000 0.10000"/>
+        <mass value="3.00000"/>
+      </inertial>
+      <visual name="mid_right_wheel">
+        <material name="Material.001"/>
+        <origin rpy="-0.00000 0.00000 0.00000" xyz="-0.00000 0.00000 0.10000"/>
+        <geometry>
+          <mesh filename="${mesh_path}/Torus.007.dae" scale="0.40000 0.40000 0.70000"/>
+        </geometry>
+      </visual>
+    </link>
+    <link name="axis_left_link">
+      <collision name="axis_left_collision">
+        <origin rpy="-1.55093 0.07494 0.77002" xyz="-0.01304 0.01116 -0.07670"/>
+        <geometry>
+          <mesh filename="${mesh_path}/Cube.005.dae" scale="0.95000 0.05000 0.10000"/>
+        </geometry>
+      </collision>
+      <inertial>
+        <inertia ixx="0.00100" ixy="-0.00000" ixz="-0.00000" iyy="0.00100" iyz="0.00000" izz="0.00100"/>
+        <origin rpy="0.00000 0.00000 0.00000" xyz="0.00000 -0.00000 0.00000"/>
+        <mass value="3.00000"/>
+      </inertial>
+      <visual name="axis_left">
+        <material name="orange"/>
+        <origin rpy="-1.55093 0.07494 0.77002" xyz="-0.00365 -0.00204 -0.05382"/>
+        <geometry>
+          <mesh filename="${mesh_path}/Cube.005.dae" scale="0.95000 0.05000 0.10000"/>
+        </geometry>
+      </visual>
+    </link>
     <link name="axis_right_link">
-    <collision name="axis_right_collision">
-      <origin rpy="1.58831 -0.01751 -0.78555" xyz="-0.02891 0.01341 -0.04021"/>
-      <geometry>
-        <mesh filename="${mesh_path}/Cube.007.dae" scale="0.95000 0.05000 0.10000"/>
-      </geometry>
-    </collision>
-    <inertial>
-      <inertia ixx="0.38352" ixy="-0.00000" ixz="0.08781" iyy="1.49498" iyz="0.00000" izz="1.11529"/>
-      <origin rpy="0.00000 0.00000 0.00000" xyz="0.00095 0.00000 -0.03832"/>
-      <mass value="3.00000"/>
-    </inertial>
-    <visual name="axis_right">
-      <material name="orange"/>
-      <origin rpy="1.58831 -0.01751 -0.78555" xyz="0.00095 0.00000 -0.03832"/>
-      <geometry>
-        <mesh filename="${mesh_path}/Cube.007.dae" scale="0.95000 0.05000 0.10000"/>
-      </geometry>
-    </visual>
-  </link>
-    <transmission name="back_left_wheel_link_joint_trans">
-        <type>transmission_interface/SimpleTransmission</type>
-        <joint name="back_left_wheel_link_joint" >
-            <hardwareInterface>hardware_interface/VelocityJointInterface</hardwareInterface>
-        </joint>
-        <actuator name="$back_left_wheel_link_joint_motor">
-            <mechanicalReduction>1</mechanicalReduction>
-        </actuator>
-    </transmission>
-    <gazebo reference="back_left_wheel_link_joint">
-        <mu1>5</mu1>
-        <mu2>5</mu2>
-        <!--kp>2.75e6</kp>
-        <kd>8.25e1</kd>
-        <fdir1>0 0 0</fdir1>
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