Commit message: moveit conf finished

File: src/rover_description/robots/robot.urdf.xacro (robot description, xacro)
@@ -24,5 +24,5 @@
 <xacro:include filename="$(find rover_description)/urdf/ros2_control.urdf.xacro"/>
 <xacro:arg name="config_controllers" default="$(find rover_description)/config/robot_controllers.yaml"/>
-<xacro:arg name="update_rate" default="100"/>
+<xacro:arg name="update_rate" default="20"/>
 <xacro:ros2_control/>
 </robot>

File: src/rover_description/urdf/arm/gripper.urdf.xacro (robot description, xacro)
@@ -1,10 +1,10 @@
 <?xml version="1.0"?>
 <robot name="gripper" xmlns:xacro="http://wiki.ros.org/xacro">
-    <xacro:macro name="gripper">
+    <xacro:macro name="gripper" params="parent *origin">
     <xacro:property name="mesh_path" value="file://$(find rover_description)/meshes/dae"/>
     <joint name="left_clamp_link_joint" type="prismatic">
         <limit lower="0.00000" upper="0.40000" effort="0.00000" velocity="0.00000"/>
         <origin rpy="-1.57080 0.00000 0.00000" xyz="0.01328 -0.34694 -0.48139"/>
-        <parent link="clamp_base_link"/>
+        <parent link="${parent}"/>
         <child link="left_clamp_link"/>
         <axis xyz="0.00000 0.00000 1.00000"/>
@@ -13,28 +13,8 @@
         <limit lower="0.00000" upper="0.40000" effort="0.00000" velocity="0.00000"/>
         <origin rpy="1.57080 0.00000 0.00000" xyz="0.01328 0.35306 -0.50058"/>
-        <parent link="clamp_base_link"/>
+        <parent link="${parent}"/>
         <child link="right_clamp_link"/>
         <axis xyz="0.00000 0.00000 1.00000"/>
     </joint>
-    <link name="clamp_base_link">
-    <collision name="clamp_base_collision">
-        <origin rpy="0.00000 0.00000 0.00000" xyz="0.00000 0.00000 -0.08713"/>
-        <geometry>
-        <mesh filename="${mesh_path}/Cylinder.005.dae" scale="0.25000 0.45000 0.05000"/>
-        </geometry>
-    </collision>
-    <inertial>
-        <inertia ixx="0.02557" ixy="-0.00000" ixz="0.00000" iyy="0.00818" iyz="-0.00000" izz="0.03291"/>
-        <origin rpy="0.00000 0.00000 0.00000" xyz="0.00000 0.00000 -0.08713"/>
-        <mass value="0.50000"/>
-    </inertial>
-    <visual name="clamp_base">
-        <material name="Material.005"/>
-        <origin rpy="0.00000 0.00000 0.00000" xyz="0.00000 0.00000 -0.08713"/>
-        <geometry>
-        <mesh filename="${mesh_path}/Cylinder.005.dae" scale="0.25000 0.45000 0.05000"/>
-        </geometry>
-    </visual>
-    </link>
     <link name="left_clamp_link">
     <collision name="left_clamp_collision">

File: src/rover_description/urdf/arm/scara.urdf.xacro (robot description, xacro)
@@ -9,10 +9,4 @@
         <child link="fixed_base_arm_link"/>
     </joint>
-    <xacro:gripper/>
-    <joint name="gripper_to_arm_joint" type="fixed">
-      <parent link="l3_arm_link"/>
-      <child link="clamp_base_link"/>
-      <origin xyz="-0.00223 -0.00306 -0.95588" rpy="0 0 0"/>
-    </joint>
     <joint name="l0_arm_link_joint" type="fixed">
         <origin rpy="0.00000 0.00000 0.00000" xyz="0.00000 0.00000 -0.04593"/>
@@ -21,5 +15,5 @@
     </joint>
     <joint name="l1_arm_link_joint" type="continuous">
-        <limit effort="0.00000" velocity="0.00000"/>
+        <limit effort="50.00000" velocity="1.50000"/>
         <origin rpy="0.00000 0.00000 0.00000" xyz="0.00000 0.00480 1.93831"/>
         <parent link="l0_arm_link"/>
@@ -28,5 +22,5 @@
     </joint>
     <joint name="l2_arm_link_joint" type="revolute">
-        <limit lower="-3.14000" upper="3.14000" effort="0.00000" velocity="0.00000"/>
+        <limit lower="-3.14000" upper="3.14000" effort="50.00000" velocity="1.50000"/>
         <origin rpy="0.00000 0.00000 1.57080" xyz="0.04172 1.09520 0.15762"/>
         <parent link="l1_arm_link"/>
@@ -35,9 +29,16 @@
     </joint>
     <joint name="l3_arm_link_joint" type="prismatic">
-        <limit lower="-2.40000" upper="0.80000" effort="0.00000" velocity="0.00000"/>
+        <limit lower="-2.40000" upper="0.80000" effort="50.00000" velocity="1.50000"/>
         <origin rpy="0.00000 0.00000 -1.57080" xyz="0.00000 -1.26247 0.09521"/>
         <parent link="l2_arm_link"/>
         <child link="l3_arm_link"/>
         <axis xyz="0.00000 0.00000 1.00000"/>
+    </joint>
+    <joint name="clamp_base_link_joint" type="continuous">
+      <limit effort="50.00000" velocity="1.50000"/>
+      <origin rpy="0.00000 0.00000 0.00000" xyz="-0.00223 -0.00306 -0.95588"/>
+      <parent link="l3_arm_link"/>
+      <child link="clamp_base_link"/>
+      <axis xyz="0.00000 0.00000 1.00000"/>
     </joint>
     <link name="fixed_base_arm_link">
@@ -141,4 +142,27 @@
     </visual>
   </link>
+  <link name="clamp_base_link">
+    <collision name="clamp_base_collision">
+        <origin rpy="0.00000 0.00000 0.00000" xyz="0.00000 0.00000 -0.08713"/>
+        <geometry>
+        <mesh filename="${mesh_path}/Cylinder.005.dae" scale="0.25000 0.45000 0.05000"/>
+        </geometry>
+    </collision>
+    <inertial>
+        <inertia ixx="0.02557" ixy="-0.00000" ixz="0.00000" iyy="0.00818" iyz="-0.00000" izz="0.03291"/>
+        <origin rpy="0.00000 0.00000 0.00000" xyz="0.00000 0.00000 -0.08713"/>
+        <mass value="0.50000"/>
+    </inertial>
+    <visual name="clamp_base">
+        <material name="Material.005"/>
+        <origin rpy="0.00000 0.00000 0.00000" xyz="0.00000 0.00000 -0.08713"/>
+        <geometry>
+        <mesh filename="${mesh_path}/Cylinder.005.dae" scale="0.25000 0.45000 0.05000"/>
+        </geometry>
+    </visual>
+  </link>
+  <xacro:gripper parent="clamp_base_link">
+    <origin rpy="0.00000 0.00000 0.00000" xyz="-0.00223 -0.00306 -0.95588"/>
+  </xacro:gripper>
 </xacro:macro>
 </robot>

File: src/rover_moveit_config/config/rover.ros2_control.xacro (robot description, xacro)
@@ -6,5 +6,5 @@
             <hardware>
                 <!-- By default, set up controllers for simulation. This won't work on real hardware -->
-                <plugin>mock_components/GenericSystem</plugin>
+                <plugin>gz_ros2_control/GazeboSimSystem</plugin>
             </hardware>
             <joint name="l1_arm_link_joint">

File: src/rover_moveit_config/config/rover.urdf.xacro (robot description, xacro)
@@ -4,6 +4,7 @@
     <!-- Import rover urdf file -->
     <xacro:include filename="$(find rover_description)/robots/robot.urdf.xacro" />
+    <xacro:include filename="rover.srdf"/>
     <!-- Import control_xacro -->
     <xacro:include filename="rover.ros2_control.xacro" />
-    <xacro:rover_ros2_control name="FakeSystem" initial_positions_file="$(arg initial_positions_file)"/>
+    <xacro:rover_ros2_control name="ScaraArm" initial_positions_file="$(arg initial_positions_file)"/>
 </robot>

Commit message: moveit funcional + camaras correctas

File: src/rover_description/robots/robot.urdf.xacro (robot description, xacro)
@@ -16,5 +16,5 @@
   </xacro:sensor_camera>
   <xacro:sensor_camera node_name="arm_camera" node_namespace="$(arg robot_ns)" frame_prefix="$(arg prefix)arm_camera_" parent="$(arg prefix)l3_arm_link" >
-          <origin xyz="0.0 0.0 -0.01" rpy="0 0 0"/>
+          <origin xyz="0.0 0.0 -1.2" rpy="0 1.57 1.57"/>
   </xacro:sensor_camera>
   <xacro:sensor_imu ns="$(arg robot_ns)" prefix="$(arg prefix)imu_" parent="$(arg prefix)base_link">

File: src/rover_description/urdf/arm/gripper.urdf.xacro (robot description, xacro)
@@ -4,5 +4,5 @@
     <xacro:property name="mesh_path" value="file://$(find rover_description)/meshes/dae"/>
     <joint name="left_clamp_link_joint" type="prismatic">
-        <limit lower="0.00000" upper="0.40000" effort="0.00000" velocity="0.00000"/>
+        <limit lower="0.00000" upper="0.40000" effort="50.00000" velocity="1.50000"/>
         <origin rpy="-1.57080 0.00000 0.00000" xyz="0.01328 -0.34694 -0.48139"/>
         <parent link="${parent}"/>
@@ -11,5 +11,5 @@
     </joint>
     <joint name="right_clamp_link_joint" type="prismatic">
-        <limit lower="0.00000" upper="0.40000" effort="0.00000" velocity="0.00000"/>
+        <limit lower="0.00000" upper="0.40000" effort="50.00000" velocity="1.50000"/>
         <origin rpy="1.57080 0.00000 0.00000" xyz="0.01328 0.35306 -0.50058"/>
         <parent link="${parent}"/>

File: src/rover_description/urdf/ros2_control.urdf.xacro (robot description, xacro)
@@ -75,4 +75,22 @@
       <state_interface name="effort"/>
     </joint>
+    <joint name="left_clamp_link_joint">
+      <command_interface name="velocity">
+        <param name="min">-10</param>
+        <param name="max">10</param>
+      </command_interface>
+      <state_interface name="position"/>
+      <state_interface name="velocity"/>
+      <state_interface name="effort"/>
+    </joint>
+    <joint name="right_clamp_link_joint">
+      <command_interface name="velocity">
+        <param name="min">-10</param>
+        <param name="max">10</param>
+      </command_interface>
+      <state_interface name="position"/>
+      <state_interface name="velocity"/>
+      <state_interface name="effort"/>
+    </joint>
     </ros2_control>
   </xacro:macro>
