Commit message: changed wheels collision

File: src/rover_description/urdf/arm/gripper.urdf.xacro (robot description, xacro)
@@ -4,5 +4,5 @@
     <xacro:property name="mesh_path" value="file://$(find rover_description)/meshes/dae"/>
     <joint name="left_clamp_link_joint" type="prismatic">
-        <limit lower="0.00000" upper="0.40000" effort="50.00000" velocity="1.50000"/>
+        <limit lower="-0.01000" upper="0.40000" effort="150.00000" velocity="1.50000"/>
         <origin rpy="-1.57080 0.00000 0.00000" xyz="0.01328 -0.34694 -0.48139"/>
         <parent link="${parent}"/>
@@ -11,5 +11,5 @@
     </joint>
     <joint name="right_clamp_link_joint" type="prismatic">
-        <limit lower="0.00000" upper="0.40000" effort="50.00000" velocity="1.50000"/>
+        <limit lower="-0.01000" upper="0.40000" effort="150.00000" velocity="1.50000"/>
         <origin rpy="1.57080 0.00000 0.00000" xyz="0.01328 0.35306 -0.50058"/>
         <parent link="${parent}"/>

File: src/rover_description/urdf/arm/scara.urdf.xacro (robot description, xacro)
@@ -15,5 +15,5 @@
     </joint>
     <joint name="l1_arm_link_joint" type="continuous">
-        <limit effort="50.00000" velocity="1.50000"/>
+        <limit effort="150.00000" velocity="2.50000"/>
         <origin rpy="0.00000 0.00000 0.00000" xyz="0.00000 0.00480 1.93831"/>
         <parent link="l0_arm_link"/>
@@ -21,6 +21,6 @@
         <axis xyz="0.00000 0.00000 1.00000"/>
     </joint>
-    <joint name="l2_arm_link_joint" type="revolute">
-        <limit lower="-3.14000" upper="3.14000" effort="50.00000" velocity="1.50000"/>
+    <joint name="l2_arm_link_joint" type="continuous">
+        <limit effort="150.00000" velocity="2.50000"/>
         <origin rpy="0.00000 0.00000 1.57080" xyz="0.04172 1.09520 0.15762"/>
         <parent link="l1_arm_link"/>
@@ -29,5 +29,5 @@
     </joint>
     <joint name="l3_arm_link_joint" type="prismatic">
-        <limit lower="-2.40000" upper="0.80000" effort="50.00000" velocity="1.50000"/>
+        <limit lower="-2.40000" upper="0.80000" effort="150.00000" velocity="2.50000"/>
         <origin rpy="0.00000 0.00000 -1.57080" xyz="0.00000 -1.26247 0.09521"/>
         <parent link="l2_arm_link"/>
@@ -36,5 +36,5 @@
     </joint>
     <joint name="clamp_base_link_joint" type="continuous">
-      <limit effort="50.00000" velocity="1.50000"/>
+      <limit effort="150.00000" velocity="2.50000"/>
       <origin rpy="0.00000 0.00000 0.00000" xyz="-0.00223 -0.00306 -0.95588"/>
       <parent link="l3_arm_link"/>

File: src/rover_description/urdf/ros2_control.urdf.xacro (robot description, xacro)
@@ -22,6 +22,6 @@
     <joint name="front_left_wheel_link_joint">
       <command_interface name="velocity">
-        <param name="min">-10</param>
-        <param name="max">10</param>
+        <param name="min">-3.14</param>
+        <param name="max">3.14</param>
       </command_interface>
       <state_interface name="position"/>
@@ -75,6 +75,44 @@
       <state_interface name="effort"/>
     </joint>
+    <!-- SCARA arm -->
+    <joint name="l1_arm_link_joint">
+      <command_interface name="position">
+        <param name="min">-3.14</param>
+        <param name="max">3.14</param>
+      </command_interface>
+      <state_interface name="position"/>
+      <state_interface name="velocity"/>
+      <state_interface name="effort"/>
+    </joint>
+    <joint name="l2_arm_link_joint">
+      <command_interface name="position">
+        <param name="min">-3.14</param>
+        <param name="max">3.14</param>
+      </command_interface>
+      <state_interface name="position"/>
+      <state_interface name="velocity"/>
+      <state_interface name="effort"/>
+    </joint>
+    <joint name="l3_arm_link_joint">
+      <command_interface name="position">
+        <param name="min">-2.4</param>
+        <param name="max">0.8</param>
+      </command_interface>
+      <state_interface name="position"/>
+      <state_interface name="velocity"/>
+      <state_interface name="effort"/>
+    </joint>
+    <joint name="clamp_base_link_joint">
+      <command_interface name="position">
+        <param name="min">-3.14</param>
+        <param name="max">3.14</param>
+      </command_interface>
+      <state_interface name="position"/>
+      <state_interface name="velocity"/>
+      <state_interface name="effort"/>
+    </joint>
+    <!-- Gripper -->
     <joint name="left_clamp_link_joint">
-      <command_interface name="velocity">
+      <command_interface name="position">
         <param name="min">-10</param>
         <param name="max">10</param>
@@ -85,5 +123,5 @@
     </joint>
     <joint name="right_clamp_link_joint">
-      <command_interface name="velocity">
+      <command_interface name="position">
         <param name="min">-10</param>
         <param name="max">10</param>

File: src/rover_description/urdf/wheels/rover_wheels.urdf.xacro (robot description, xacro)
@@ -54,5 +54,5 @@
     </link>
     <joint name="back_left_wheel_link_joint" type="continuous">
-      <limit effort="50.0" velocity="20.0"/>
+      <limit effort="100.0" velocity="20.0"/>
       <dynamics damping="0.05" friction="0.1"/>
       <origin rpy="-0.03655 0.06700 -0.01743" xyz="-1.43329 -0.48979 0.41533"/>
@@ -62,5 +62,5 @@
     </joint>
     <joint name="front_left_wheel_link_joint" type="continuous">
-      <limit effort="50.0" velocity="20.0"/>
+      <limit effort="100.0" velocity="20.0"/>
       <dynamics damping="0.05" friction="0.1"/>
       <origin rpy="-0.03655 0.06700 -0.01743" xyz="1.55952 -0.54195 0.21447"/>
@@ -70,5 +70,5 @@
     </joint>
     <joint name="mid_left_wheel_link_joint" type="continuous">
-      <limit effort="50.0" velocity="20.0"/>
+      <limit effort="100.0" velocity="20.0"/>
       <dynamics damping="0.05" friction="0.1"/>
       <origin rpy="-0.03655 0.06700 -0.01743" xyz="0.06311 -0.51587 0.31490"/>
@@ -78,5 +78,5 @@
     </joint>
     <joint name="back_right_wheel_link_joint" type="continuous">
-      <limit effort="50.0" velocity="20.0"/>
+      <limit effort="100.0" velocity="20.0"/>
       <dynamics damping="0.05" friction="0.1"/>
       <origin rpy="3.14159 -0.02477 -0.00000" xyz="-1.45614 0.52600 0.26402"/>
@@ -86,5 +86,5 @@
     </joint>
     <joint name="front_right_wheel_link_joint" type="continuous">
-      <limit effort="50.0" velocity="20.0"/>
+      <limit effort="100.0" velocity="20.0"/>
       <dynamics damping="0.05" friction="0.1"/>
       <origin rpy="3.14159 -0.02477 -0.00000" xyz="1.54294 0.52600 0.33832"/>
@@ -94,5 +94,5 @@
     </joint>
     <joint name="mid_right_wheel_link_joint" type="continuous">
-      <limit effort="50.0" velocity="20.0"/>
+      <limit effort="100.0" velocity="20.0"/>
       <dynamics damping="0.05" friction="0.1"/>
       <origin rpy="3.14159 -0.02477 -0.00000" xyz="0.04340 0.52600 0.30117"/>
@@ -105,5 +105,5 @@
         <origin rpy="-0.00497 -0.00000 0.00000" xyz="-0.00000 0.00042 -0.12869"/>
         <geometry>
-          <mesh filename="${mesh_path}/Torus.005.dae" scale="0.40000 0.40000 0.70000"/>
+          <cylinder length="0.2" radius="0.5"/>
         </geometry>
       </collision>
@@ -125,5 +125,5 @@
         <origin rpy="-0.00497 -0.00000 0.00000" xyz="0.00000 0.00043 -0.12796"/>
         <geometry>
-          <mesh filename="${mesh_path}/Torus.009.dae" scale="0.40000 0.40000 0.70000"/>
+          <cylinder length="0.2" radius="0.5"/>
         </geometry>
       </collision>
@@ -145,5 +145,5 @@
         <origin rpy="-0.00497 -0.00000 0.00000" xyz="0.00000 0.00042 -0.12869"/>
         <geometry>
-          <mesh filename="${mesh_path}/Torus.006.dae" scale="0.40000 0.40000 0.70000"/>
+          <cylinder length="0.2" radius="0.5"/>
         </geometry>
       </collision>
@@ -165,5 +165,5 @@
         <origin rpy="-3.14159 0.00000 0.00000" xyz="-0.00000 0.00000 0.10000"/>
         <geometry>
-          <mesh filename="${mesh_path}/Torus.dae" scale="0.40000 0.40000 0.70000"/>
+          <cylinder length="0.2" radius="0.5"/>
         </geometry>
       </collision>
@@ -185,5 +185,5 @@
         <origin rpy="-3.14159 0.00000 0.00000" xyz="0.00000 0.00000 0.10000"/>
         <geometry>
-          <mesh filename="${mesh_path}/Torus.008.dae" scale="0.40000 0.40000 0.70000"/>
+          <cylinder length="0.2" radius="0.5"/>
         </geometry>
       </collision>
@@ -205,5 +205,5 @@
         <origin rpy="-3.14159 0.00000 0.00000" xyz="-0.00000 0.00000 0.11498"/>
         <geometry>
-          <mesh filename="${mesh_path}/Torus.007.dae" scale="0.40000 0.40000 0.70000"/>
+          <cylinder length="0.2" radius="0.5"/>
         </geometry>
       </collision>
