Commit message: modificaciones

File: src/rover_description/urdf/arm/scara.urdf.xacro (robot description, xacro)
@@ -15,5 +15,5 @@
     </joint>
     <joint name="l1_arm_link_joint" type="continuous">
-        <limit effort="150.00000" velocity="2.50000"/>
+        <limit effort="150.00000" velocity="3.00000"/>
         <origin rpy="0.00000 0.00000 0.00000" xyz="0.00000 0.00480 1.93831"/>
         <parent link="l0_arm_link"/>
@@ -22,5 +22,5 @@
     </joint>
     <joint name="l2_arm_link_joint" type="continuous">
-        <limit effort="150.00000" velocity="2.50000"/>
+        <limit effort="150.00000" velocity="3.00000"/>
         <origin rpy="0.00000 0.00000 1.57080" xyz="0.04172 1.09520 0.15762"/>
         <parent link="l1_arm_link"/>
@@ -29,5 +29,5 @@
     </joint>
     <joint name="l3_arm_link_joint" type="prismatic">
-        <limit lower="-2.40000" upper="0.80000" effort="150.00000" velocity="2.50000"/>
+        <limit lower="-2.40000" upper="0.80000" effort="150.00000" velocity="3.00000"/>
         <origin rpy="0.00000 0.00000 -1.57080" xyz="0.00000 -1.26247 0.09521"/>
         <parent link="l2_arm_link"/>
@@ -36,5 +36,5 @@
     </joint>
     <joint name="clamp_base_link_joint" type="continuous">
-      <limit effort="150.00000" velocity="2.50000"/>
+      <limit effort="150.00000" velocity="3.00000"/>
       <origin rpy="0.00000 0.00000 0.00000" xyz="-0.00223 -0.00306 -0.95588"/>
       <parent link="l3_arm_link"/>

File: src/rover_description/urdf/sensors/camera.urdf.xacro (robot description, xacro)
@@ -16,4 +16,10 @@
       </inertial>
     </link>
+    <joint name="${frame_prefix}camera_optical_joint" type="fixed">
+      <origin xyz="0 0 0" rpy="-1.5707963267948966 0 -1.5707963267948966"/>
+      <parent link="${frame_prefix}camera_frame"/>
+      <child link="${frame_prefix}camera_optical_frame"/>
+    </joint>
+    <link name="${frame_prefix}camera_optical_frame"/>
     <gazebo reference="${frame_prefix}camera_frame">
       <sensor name="${frame_prefix}sensor" type="camera">
@@ -21,4 +27,5 @@
         <visualize>true</visualize>
         <update_rate>30</update_rate>
+        <gz_frame_id>${frame_prefix}camera_optical_frame</gz_frame_id>
         <topic>${node_namespace}/${node_name}/image</topic>
         <camera>

File: src/rover_moveit_config/config/rover.urdf.xacro (robot description, xacro)
@@ -1,10 +1,5 @@
 <?xml version="1.0"?>
 <robot xmlns:xacro="http://www.ros.org/wiki/xacro" name="rover">
-    <xacro:arg name="initial_positions_file" default="initial_positions.yaml" />
     <!-- Import rover urdf file -->
     <xacro:include filename="$(find rover_description)/robots/robot.urdf.xacro" />
-    <xacro:include filename="rover.srdf"/>
-    <!-- Import control_xacro -->
-    <xacro:include filename="rover.ros2_control.xacro" />
-    <xacro:rover_ros2_control name="ScaraArm" initial_positions_file="$(arg initial_positions_file)"/>
 </robot>
